File: V4/Hw/Magspoof_V4.kicad_sch (KiCad schematic)
At the start: 35 parts, among them J1 Coil, J2 SWD, P1 USB_C_Plug_USB2.0, Q1 DMG3415U-7, SW1 ON, SW3 S1, SW4 SOURCE MAG, SW5 RESET, U1 CH552G, U2 AP2112K-3.3, U3 TC4424, U5 MCP73831

Commit message: change DFN-8 to SOIC-8 TC4424 and add 3d model of SW1,4
Parts:
- U3: footprint Library:TC4424EMF(v3) -> Package_SO:SOIC-8_3.9x4.9mm_P1.27mm
Changed lines of the file:
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@@
       (effects (font (size 1.524 1.524)))
     )
-    (property "Footprint" "Library:TC4424EMF(v3)" (at 216.789 77.216 0)
+    (property "Footprint" "Package_SO:SOIC-8_3.9x4.9mm_P1.27mm" (at 216.789 77.216 0)
       (effects (font (size 1.524 1.524)) hide)
     )
@@
       (effects (font (size 1.27 1.27)) hide)
     )
+    (pin "2")
     (pin "3")
-    (pin "2")
-    (instances
-      (project "Magspoof_V4"
+    (instances
+      (project "Magspoof_V4"

Commit message: Update BOM
Parts:
- D4: Proveedor MOUSER -> LCSC; manf# 150080GS75000 -> D-R080508L3-KS2
- U3: Proveedor MOUSER -> LCSC
- U5: LCSC# C38066 -> C14879; Proveedor MOUSER -> LCSC
Changed lines of the file:
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@@
       (effects (font (size 1.27 1.27)) hide)
     )
-    (property "Proveedor" "MOUSER" (at 216.789 77.216 0)
+    (property "Proveedor" "LCSC" (at 216.789 77.216 0)
       (effects (font (size 1.27 1.27)) hide)
     )
@@
       (effects (font (size 1.27 1.27)) hide)
     )
-    (property "Proveedor" "MOUSER" (at 228.854 27.686 0)
-      (effects (font (size 1.27 1.27)) hide)
-    )
-    (property "LCSC#" "C38066" (at 228.854 27.686 0)
+    (property "Proveedor" "LCSC" (at 228.854 27.686 0)
+      (effects (font (size 1.27 1.27)) hide)
+    )
+    (property "LCSC#" "C14879" (at 228.854 27.686 0)
       (effects (font (size 1.27 1.27)) hide)
     )
@@
       (effects (font (size 1.27 1.27)) hide)
     )
-    (property "Datasheet" "https://www.mouser.mx/datasheet/2/60/js-1841892.pdf" (at 85.725 36.957 0)
+    (property "Datasheet" "https://datasheet.lcsc.com/lcsc/1808041445_ALPSALPINE-SSSS811101_C109335.pdf" (at 85.725 36.957 0)
       (effects (font (size 1.27 1.27)) hide)
     )
@@
       (effects (font (size 1.27 1.27)) hide)
     )
-    (property "manf#" "150080GS75000" (at 337.947 153.797 0)
-      (effects (font (size 1.27 1.27)) hide)
-    )
-    (property "Proveedor" "MOUSER" (at 243.713 44.45 0)
+    (property "manf#" "D-R080508L3-KS2" (at 337.947 153.797 0)
+      (effects (font (size 1.27 1.27)) hide)
+    )
+    (property "Proveedor" "LCSC" (at 243.713 44.45 0)
       (effects (font (size 1.27 1.27)) hide)
     )
@@
       (effects (font (size 1.27 1.27)) hide)
     )
-    (property "Datasheet" "https://www.mouser.mx/datasheet/2/60/js-1841892.pdf" (at 239.649 73.406 0)
+    (property "Datasheet" "https://datasheet.lcsc.com/lcsc/1808041445_ALPSALPINE-SSSS811101_C109335.pdf" (at 239.649 73.406 0)
       (effects (font (size 1.27 1.27)) hide)
     )
@@
     )
     (property "LCSC#" "C109335" (at 239.649 73.406 0)
-      (effects (font (size 1.27 1.27)) hide)
-    )
-    (property "Campo7" "" (at 239.649 73.406 90)
       (effects (font (size 1.27 1.27)) hide)
     )
@@
       (effects (font (size 1.27 1.27)) hide)
     )
-    (property "Datasheet" "https://www.mouser.mx/datasheet/2/427/mfuserie-1762582.pdf" (at 45.339 30.48 0)
-      (effects (font (size 1.27 1.27)) hide)
-    )
+    (property "Datasheet" "https://datasheet.lcsc.com/lcsc/1809211126_Shenzhen-JDT-Fuse-JFC0603-0500FS_C136327.pdf" (at 45.339 30.48 0)
+      (effects (font (size 1.27 1.27)) hide)
+    )

Commit message: Update BOM (jlcpcb components)
Parts:
- F1: manf# (none) -> JFC0603-0500FS
- R1, R11, R7: Proveedor MOUSER -> LCSC
- R10: Proveedor MOUSER -> LCSC; manf# SFR01MZPJ471 -> RC0402FR-07470RL
- R2, R3, R9: LCSC# C2692696 -> C317922; manf# PTFR0402B5K10P9 -> HP02WAF2002TCE
- SW1, SW4: manf# (none) -> SSSS811101
- U1: manf# (none) -> CH552G
- U2: LCSC# C150742 -> C47773; Proveedor (none) -> LCSC; manf# AP7347DQ-33W5-7 -> RT9013-33GB
- U5: LCSC# C14879 -> C424093; manf# MCP73831T-5ACI/OT -> MCP73831T-2ACI/OT
Changed lines of the file:
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@@
+      (effects (font (size 1.27 1.27)) hide)
+    )
+    (property "manf#" "CH552G" (at 70.231 96.52 0)
       (effects (font (size 1.27 1.27)) hide)
     )
@@
       (effects (font (size 1.27 1.27)) hide)
     )
-    (property "LCSC#" "C2692696" (at 49.022 38.1 0)
-      (effects (font (size 1.27 1.27)) hide)
-    )
-    (property "manf#" "PTFR0402B5K10P9" (at 49.022 38.1 0)
+    (property "LCSC#" "C317922" (at 49.022 38.1 0)
+      (effects (font (size 1.27 1.27)) hide)
+    )
+    (property "manf#" "HP02WAF2002TCE" (at 49.022 38.1 0)
       (effects (font (size 1.27 1.27)) hide)
     )
@@
       (effects (font (size 1.27 1.27)) hide)
     )
-    (property "manf#" "MCP73831T-5ACI/OT\n" (at 228.854 27.686 0)
+    (property "manf#" "MCP73831T-2ACI/OT" (at 228.854 27.686 0)
       (effects (font (size 1.27 1.27)) hide)
     )
@@
       (effects (font (size 1.27 1.27)) hide)
     )
-    (property "LCSC#" "C14879" (at 228.854 27.686 0)
+    (property "LCSC#" "C424093" (at 228.854 27.686 0)
       (effects (font (size 1.27 1.27)) hide)
     )
@@
       (effects (font (size 1.27 1.27)) hide)
     )
-    (property "LCSC#" "C2692696" (at 44.323 35.56 0)
-      (effects (font (size 1.27 1.27)) hide)
-    )
-    (property "manf#" "PTFR0402B5K10P9" (at 44.323 35.56 0)
+    (property "LCSC#" "C317922" (at 44.323 35.56 0)
+      (effects (font (size 1.27 1.27)) hide)
+    )
+    (property "manf#" "HP02WAF2002TCE" (at 44.323 35.56 0)
       (effects (font (size 1.27 1.27)) hide)
     )
@@
       (effects (font (size 1.27 1.27)) hide)
     )
-    (property "Proveedor" "MOUSER" (at 107.061 107.442 0)
+    (property "Proveedor" "LCSC" (at 107.061 107.442 0)
       (effects (font (size 1.27 1.27)) hide)
     )
@@
       (effects (font (size 1.27 1.27)) hide)
     )
-    (property "manf#" "AP7347DQ-33W5-7" (at 109.22 39.497 0)
-      (effects (font (size 1.27 1.27)) hide)
-    )
-    (property "LCSC#" "C150742" (at 109.22 39.497 0)
+    (property "manf#" "RT9013-33GB" (at 109.22 39.497 0)
+      (effects (font (size 1.27 1.27)) hide)
+    )
+    (property "LCSC#" "C47773" (at 109.22 39.497 0)
+      (effects (font (size 1.27 1.27)) hide)
+    )
+    (property "Proveedor" "LCSC" (at 109.22 39.497 0)
       (effects (font (size 1.27 1.27)) hide)
     )
@@
       (effects (font (size 1.27 1.27)) hide)
     )
-    (property "LCSC#" "C2692696" (at 134.366 122.174 0)
-      (effects (font (size 1.27 1.27)) hide)
-    )
-    (property "manf#" "PTFR0402B5K10P9" (at 213.233 36.195 0)
+    (property "LCSC#" "C317922" (at 134.366 122.174 0)
+      (effects (font (size 1.27 1.27)) hide)
+    )
+    (property "manf#" "HP02WAF2002TCE" (at 213.233 36.195 0)
       (effects (font (size 1.27 1.27)) hide)
     )
@@
       (effects (font (size 1.27 1.27)) hide)
     )
-    (property "Proveedor" "MOUSER" (at 147.32 43.053 0)
+    (property "Proveedor" "LCSC" (at 147.32 43.053 0)
       (effects (font (size 1.27 1.27)) hide)
     )
@@
       (effects (font (size 1.27 1.27)) hide)
     )
-    (property "manf#" "SFR01MZPJ471" (at 134.366 121.158 0)
-      (effects (font (size 1.27 1.27)) hide)
-    )
-    (property "Proveedor" "MOUSER" (at 243.713 35.687 0)
+    (property "manf#" "RC0402FR-07470RL" (at 134.366 121.158 0)
+      (effects (font (size 1.27 1.27)) hide)
+    )
+    (property "Proveedor" "LCSC" (at 243.713 35.687 0)
       (effects (font (size 1.27 1.27)) hide)
     )
@@
       (effects (font (size 1.27 1.27)) hide)
     )
-    (property "manf#" "" (at 85.725 36.957 0)
+    (property "manf#" "SSSS811101" (at 85.725 36.957 0)
       (effects (font (size 1.27 1.27)) hide)
     )
@@
       (effects (font (size 1.27 1.27)) hide)
     )
-    (property "Proveedor" "MOUSER" (at 65.532 43.688 0)
+    (property "Proveedor" "LCSC" (at 65.532 43.688 0)
       (effects (font (size 1.27 1.27)) hide)
     )
@@
       (effects (font (size 1.27 1.27)) hide)
     )
-    (property "manf#" "" (at 239.649 73.406 0)
+    (property "manf#" "SSSS811101" (at 239.649 73.406 0)
       (effects (font (size 1.27 1.27)) hide)
     )
@@
       (effects (font (size 1.27 1.27)) hide)
     )
-    (property "manf#" "" (at 45.339 30.48 0)
-      (effects (font (size 1.27 1.27)) hide)
-    )
+    (property "manf#" "JFC0603-0500FS" (at 45.339 30.48 0)
+      (effects (font (size 1.27 1.27)) hide)
+    )
